Commit message: robotu gazeboda kontrol etmek

File: description/robot_core.xacro (robot description, xacro)
@@ -41,4 +41,7 @@
             <origin xyz="0.15 0 0.075" rpy="0 0 0"/>
         </xacro:inertial_box>
+        <gazebo reference="chassis">
+            <material>Gazebo/Yellow</material>
+        </gazebo>
     </link>
     <!-- LEFT WHEEL LINK-->
@@ -65,4 +68,7 @@
         </xacro:inertial_cylinder>
     </link>
+    <gazebo reference="left_wheel">
+            <material>Gazebo/Red</material>
+        </gazebo>
     <!-- RIGHT WHEEL LINK-->
     <joint name="right_wheel_joint" type="continuous">
@@ -88,4 +94,7 @@
         </xacro:inertial_cylinder>
     </link>
+    <gazebo reference="right_wheel">
+            <material>Gazebo/Red</material>
+        </gazebo>
     <!-- CASTER WHEEL LINK-->
     <joint name="caster_wheel_joint" type="fixed">
@@ -111,3 +120,8 @@
         </xacro:inertial_sphere>
     </link>
+    <gazebo reference="caster_wheel">
+        <material>Gazebo/Black</material>
+        <mu1 value="0.001"/>
+        <mu2 value="0.001"/>
+        </gazebo>
 </robot>

Commit message: Lidarın eklenmesi

File: description/robot_core.xacro (robot description, xacro)
@@ -13,4 +13,7 @@
     <material name="black">
         <color rgba="0 0 0 1"/>
+    </material>
+    <material name="red">
+        <color rgba="1 0 0 1"/>
     </material>
     <!--BASE LINK -->
@@ -42,5 +45,5 @@
         </xacro:inertial_box>
         <gazebo reference="chassis">
-            <material>Gazebo/Yellow</material>
+            <material>Gazebo/White</material>
         </gazebo>
     </link>
